File: SC_lab/Projects/Elmo_nine_FET/FET_Mux/FET_mux_2layer.brd (EAGLE design)
At the start: 48.2 x 45.4 mm, 11 parts

Commit message: edit  fet project
Routing:
- net N$1: track 0.00 -> 2.41 mm
- net P05: track 7.91 -> 10.1 mm
- net N$2: track 0.00 -> 2.03 mm
- net N$3: track 0.00 -> 1.83 mm
- net GND: track 22.4 -> 23.9 mm
- net N$8: track 0.00 -> 1.07 mm
- net N$7: track 0.00 -> 1.07 mm
- net N$5: track 0.00 -> 0.89 mm
- net N$4: track 0.00 -> 0.89 mm
- net N$6: track 0.00 -> 0.56 mm
